File: PCB/anchor/anchor.kicad_sch (KiCad schematic)
At the start: 15 parts, among them J1 Conn_ARM_SWD_TagConnect_TC203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, J2 Conn_ARM_JTAG_SWD_10, J3 SM02B-SRSS-TB LFSN, U1 Voltage Regulator, U2 DWM3001C UWB, U3 LYR998

Commit message: Tag and Anchor schematic updates
Parts:
- removed J1: Conn_ARM_SWD_TagConnect_TC2030-NL, Connector:Tag-Connect_TC2030-IDC-NL_2x03_P1.27mm_Vertical, symbol Connector:Conn_ARM_SWD_TagConnect_TC2030-NL
- removed TP1: DWM Test Point, symbol Connector:TestPoint
- added C7: 10uF, symbol Device:C
- added C8: 100nF, symbol Device:C
- added D1: LTST-C235KGKRKT, LED_SMD:LED_LiteOn_LTST-C235KGKRKT, symbol LED:LTST-C235KGKRKT
- added D2, D3: LED, symbol Device:LED
- added J1, J4, J5, J6, J7, J8: TSM-102-01-X-SV, TSM-102-01-X-SV:SAMTEC_TSM-102-01-X-SV, symbol sdp:TSM-102-01-X-SV
- added Q1, Q2: IRLML2402TRPBF, digikey-footprints:SOT-23-3, symbol dk_Transistors-FETs-MOSFETs-Single:IRLML2402TRPBF
- added R1, R3: 1K5, symbol Device:R_US
- added R2, R4: 100K, symbol Device:R_US
- added R5: 150, symbol Device:R_US
- added R6: 820, symbol Device:R_US
- added R7, R8: 1k8, symbol Device:R_US
- added S1: TL3315NF160Q, digikey-footprints:Switch_Tactile_SMD_4.5x4.5mm_TL3315NF160Q, symbol dk_Tactile-Switches:TL3315NF160Q
- added TP2, TP3: TestPoint, symbol Connector:TestPoint
Connections:
- net RESET is gone; now on net RST: J2.10 (~{RESET}), U2.47 (RESET)
- net GND: now also U2.12 (VDD), U3.5 (GND), C7.1, C7.2, C8.1, C8.2, J6.01, J7.02, R2.2, R4.2, S1.3, S1.4, TP3.1
- net Vreg: now also J1.02, J4.01, J7.01, J8.01, R5.1, R6.1; no longer B1.1, B1.2, B2.2, C3.1, C4.1, C5.1, C6.1, U2.12 (VDD)
- net SWD_CLK: now reaches J2.4 (SWCLK/TCK), U2.2 (SWD_CLK)
- net SWD_DIO: now reaches J2.2 (SWDIO/TMS), U2.3 (SWD_DIO)
- net RX: now reaches U2.32 (P0.15)
- net RX: now also U3.4 (TXD)
- net TX: now reaches U2.34 (P0.19)
- net TX: now also U3.3 (RXD)
- net at U2.44 (DW_GP3): now also R1.1
- net at U2.45 (DW_GP2): now also R3.1
- net at U2.6 (P0.17): now also R8.2
- net at U2.7 (P0.14): now also R7.2
- net at U1.1 (IN), U1.3 (EN): now also J5.02; no longer J3.1
- net at U3.1 (VDD): now also B1.1, B1.2, B2.2, C3.1, C4.1, C5.1, C6.1, J4.02
- net RST: now reaches U3.2 (NRST)
- net RST: now also S1.1, S1.2
- new net: D3.1 (K), R8.1
- new net: D3.2 (A), J8.02
- new net: Q2.1 (G), R3.2, R4.1
- new net: D1.1 (K2), Q1.3 (D)
- new net: D1.2 (A2), R5.2
- new net: D1.3 (A1), R6.2
- new net: D1.4 (K1), Q2.3 (D)
- new net: Q1.1 (G), R1.2, R2.1
- new net: J6.02, Q1.2 (S), Q2.2 (S)
- new net: D2.1 (K), R7.1
- new net: D2.2 (A), J1.01
- new net: J3.1, J5.01, TP2.1
- no-connect marks 42 -> 35
Other:
- note added: "LoRa Module"
- note added: "Programming Connector"
- note added: "Qorvo Combo Module and Test Peripherals"
- note added: "Vin and Voltage Regulator"
- title: (none) -> BareTag_Anchor
- moved on the sheet: B1, B2, C1, C2, C3, C4, C5, C6, J2, J3, U1, U2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
