File: PCB/tag/tag/tag.kicad_sch (KiCad schematic)
At the start: 30 parts, among them J1 SM02B-SRSS-TB LFSN, J2 Conn_ARM_SWD_TagConnect_TC203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, J3 Conn_ARM_JTAG_SWD_10, J4 TSM-102-01-X-SV, J5 TSM-102-01-X-SV, J6 TSM-102-01-X-SV, J7 TSM-102-01-X-SV, Q1 IRLML2402TRPBF, Q2 IRLML2402TRPBF, U1 DWM3001C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

Commit message: final tag
Parts:
- C3: footprint (none) -> Capacitor_SMD:C_0603_1608Metric
- C4: footprint (none) -> imported:GRM155C80J225KE95D
- D1: value LTST-C235KGKRKT -> APHBM2012LSURKSYKC; footprint LED_SMD:LED_LiteOn_LTST-C235KGKRKT -> imported:LED_APHBM2012LSURKSYKC
- D2, D3: footprint (none) -> imported:WL-SMCW_0603
- J2: footprint Connector:Tag-Connect_TC2030-IDC-NL_2x03_P1.27mm_Vertical -> (none)
- J4, J5, J6, J7: footprint TSM-102-01-X-SV:SAMTEC_TSM-102-01-X-SV -> imported:SAMTEC_TSM-102-01-X-SV
- R1, R2, R3, R4, R5, R6, R7, R8: footprint (none) -> Resistor_SMD:R_0402_1005Metric
- TP1: value TestPoint -> Vgnd; footprint (none) -> TestPoint:TestPoint_Pad_D1.0mm
- TP2: value TestPoint -> Vbatt; footprint (none) -> TestPoint:TestPoint_Pad_D1.0mm
- TP3: value TestPoint -> Vreg; footprint (none) -> TestPoint:TestPoint_Pad_D1.0mm
Connections:
- net 3001vdd: now reaches C3.1, C4.1, J4.02, U1.12 (VDD)
- net LED GPIO Wires: no longer names the net of R7.2, U1.7 (P0.14)
Changed lines of the file:
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@@
 		(rev "1")
 		(company "SDP Team 3")
-		(comment 1 "Authors: Connor McGarry and Sean Brown")
+		(comment 1 "Authors: Connor McGarry, Sean Brown, Walter Tebbetts, Ken Su")
 	)
 	(junction
@@
 		)
 	)
-	(label "LED GPIO Wires"
-		(at 147.32 69.85 180)
-		(fields_autoplaced yes)
-		(effects
-			(font
-				(size 1.27 1.27)
-			)
-			(justify right bottom)
-		)
-	)
 	(label "Vreg +3.3V"
 		(at 31.75 52.07 270)
@@
 		)
 	)
+	(label "3001vdd"
+		(at 125.73 105.41 0)
+		(fields_autoplaced yes)
+		(effects
+			(font
+				(size 1.27 1.27)
+			)
+			(justify left bottom)
+		)
+	)
 	(label "RST"
 		(at 224.79 57.15 180)
@@
 			)
 		)
-		(property "Footprint" ""
+		(property "Footprint" "Resistor_SMD:R_0402_1005Metric"
 			(at 261.366 59.944 90)
 			(effects
@@
 			)
 		)
-		(property "Value" "TestPoint"
+		(property "Value" "Vgnd"
 			(at 20.574 180.34 90)
 			(effects
@@
 			)
 		)
-		(property "Footprint" ""
+		(property "Footprint" "TestPoint:TestPoint_Pad_D1.0mm"
 			(at 27.94 171.45 0)
 			(effects
@@
 			)
 		)
-		(property "Footprint" ""
+		(property "Footprint" "imported:GRM155C80J225KE95D"
 			(at 125.4252 113.03 0)
 			(effects
@@
 			)
 		)
-		(property "Footprint" ""
+		(property "Footprint" "Resistor_SMD:R_0402_1005Metric"
 			(at 234.696 127.254 90)
 			(effects
@@
 			)
 		)
-		(property "Footprint" ""
+		(property "Footprint" "Resistor_SMD:R_0402_1005Metric"
 			(at 130.556 63.754 90)
 			(effects
@@
 			)
 		)
-		(property "Footprint" ""
+		(property "Footprint" "Resistor_SMD:R_0402_1005Metric"
 			(at 230.886 127.254 90)
 			(effects
@@
 			)
 		)
-		(property "Footprint" "TSM-102-01-X-SV:SAMTEC_TSM-102-01-X-SV"
+		(property "Footprint" "imported:SAMTEC_TSM-102-01-X-SV"
 			(at 255.524 136.906 0)
 			(effects
@@
 			)
 		)
-		(property "Footprint" ""
+		(property "Footprint" "Capacitor_SMD:C_0603_1608Metric"
 			(at 136.8552 113.03 0)
 			(effects
@@
 			)
 		)
-		(property "Footprint" "Connector:Tag-Connect_TC2030-IDC-NL_2x03_P1.27mm_Vertical"
+		(property "Footprint" ""
 			(at 72.39 95.25 0)
 			(effects
@@
 			)
 		)
-		(property "Datasheet" "https://www.tag-connect.com/wp-content/uploads/bsk-pdf-manager/TC2030-CTX_1.pdf"
+		(property "Datasheet" "https://www.tag-connect.com/wp-content/uploads/bsk-pdf-manager/2020/12/EC-6Pin_7_9.pdf"
 			(at 72.39 92.71 0)
 			(effects
@@
 			)
 		)
-		(property "Value" "TestPoint"
+		(property "Value" "Vbatt"
 			(at 20.828 170.434 90)
 			(effects
@@
 			)
 		)
-		(property "Footprint" ""
+		(property "Footprint" "TestPoint:TestPoint_Pad_D1.0mm"
 			(at 27.94 168.91 0)
 			(effects
@@
 			)
 		)
-		(property "Footprint" "TSM-102-01-X-SV:SAMTEC_TSM-102-01-X-SV"
+		(property "Footprint" "imported:SAMTEC_TSM-102-01-X-SV"
 			(at 110.744 49.276 0)
 			(effects
@@
 			)
 		)
-		(property "Value" "TestPoint"
-			(at 126.492 163.068 0)
+		(property "Value" "Vreg"
+			(at 128.27 162.814 0)
 			(effects
 				(font
@@
 			)
 		)
-		(property "Footprint" ""
+		(property "Footprint" "TestPoint:TestPoint_Pad_D1.0mm"
 			(at 135.89 168.91 0)
 			(effects
@@
 			)
 		)
-		(property "Footprint" ""
+		(property "Footprint" "imported:WL-SMCW_0603"
 			(at 120.65 50.8 0)
 			(effects
@@
 			)
 		)
-		(property "Footprint" ""
+		(property "Footprint" "Resistor_SMD:R_0402_1005Metric"
 			(at 234.696 73.914 90)
 			(effects
@@
 			)
 		)
-		(property "Footprint" "TSM-102-01-X-SV:SAMTEC_TSM-102-01-X-SV"
+		(property "Footprint" "imported:SAMTEC_TSM-102-01-X-SV"
 			(at 139.446 37.084 0)
 			(effects
@@
 			)
 		)
-		(property "Footprint" ""
+		(property "Footprint" "Resistor_SMD:R_0402_1005Metric"
 			(at 121.666 63.754 90)
 			(effects
@@
 			)
 		)
-		(property "Footprint" ""
+		(property "Footprint" "imported:WL-SMCW_0603"
 			(at 129.54 50.8 0)
 			(effects
@@
 			)
 		)
-		(property "Footprint" ""
+		(property "Footprint" "Resistor_SMD:R_0402_1005Metric"
 			(at 266.446 59.944 90)
 			(effects
@@
 			)
 		)
-		(property "Value" "LTST-C235KGKRKT"
+		(property "Value" "APHBM2012LSURKSYKC"
 			(at 254.508 67.31 90)
 			(effects
@@
 			)
 		)
-		(property "Footprint" "LED_SMD:LED_LiteOn_LTST-C235KGKRKT"
+		(property "Footprint" "imported:LED_APHBM2012LSURKSYKC"
 			(at 262.89 75.692 0)
 			(effects
@@
 			)
 		)
-		(property "Datasheet" "https://optoelectronics.liteon.com/upload/download/DS22-2009-0219/LTST-C235KGKRKT.pdf"
+		(property "Datasheet" ""
 			(at 262.89 75.692 0)
 			(effects
@@
 			)
 		)
-		(property "Footprint" ""
+		(property "Footprint" "Resistor_SMD:R_0402_1005Metric"
 			(at 230.886 73.914 90)
 			(effects
@@
 			)
 		)
-		(property "Footprint" "TSM-102-01-X-SV:SAMTEC_TSM-102-01-X-SV"
+		(property "Footprint" "imported:SAMTEC_TSM-102-01-X-SV"
 			(at 110.744 95.504 0)
 			(effects
