File: PCB/tag/tagv2/tagv2.kicad_sch (KiCad schematic)
At the start: 20 parts, among them J1 SM02B-SRSS-TB LFSN, J2 Conn_ARM_SWD_TagConnect_TC203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, J3 Conn_ARM_JTAG_SWD_10, J4 PRT-12807, Q1 IRLML2402TRPBF, Q2 IRLML2402TRPBF, U1 DWM3001C, U2 TPS79933DDCR

Commit message: new pcb
Parts:
- removed J4: PRT-12807, imported:2*3male, symbol imported:PRT-12807
- added J5: 54202-T0804LF, imported:AMPHENOL_54202-T0804LF, symbol imported:54202-T0804LF
Connections:
- net GND: now also J5.B1
- net RST: now also J5.A2
- net RX: now also J5.A4
- net SDA: now also J5.B3
- net SLC: now also J5.B4
- net TX: now also J5.A3
- net Vbat +3.7V: now also J5.A1
- net wakeup: now also J5.B2
- net at R5.2: now also D1.1 (A2); no longer D1.2 (A2)
- net at Q1.3 (D): now also D1.2 (K2); no longer D1.1 (K2)
- net at Q2.3 (D): now also D1.3 (K1); no longer D1.4 (K1)
- net at R6.2: now also D1.4 (A1); no longer D1.3 (A1)
Other:
- note added: "Debugging Header"
