File: PCB/donglev1-2025-02-02_151608/donglev1.kicad_pcb (KiCad board)
At the start: 2 copper layers, 16.6 x 21.5 mm, 15 parts, among them IC1 CP2102N-24, J1 Conn_01x05, J2 USB_A

Commit message: other firmware testing
Parts:
- removed J2: USB_A, Adafruit CP2102N Friend:17340281
- added J1: 1734028-1, Connector_USB:USB_A_CNCTech_1001-011-01101_Horizontal, F.Cu at (127.7, 70.3)
- C1, C4: value 0.1uF -> C0603C104J4RACTU
- C2, C3, C5: value 10uF -> C0603C106M9PAC7867
- D1: renamed from D2; value GREEN -> D1
- D2: renamed from D1; value RED -> D2
- R1, R2, R6: value 20K -> RT0603BRD0720KL
- R5: value 47K -> RC0603FR-0747KL
- U1: renamed from IC1; footprint Adafruit CP2102N Friend:QFN24_CP2102N_SIL -> Adafruit CP2102N Friend:QFN24_CP2102N_SIL-L
- U2: renamed from J1; value Conn_01x05 -> RYLR998
Connections:
- D1 pad A: Net-(D2-PadA) -> (no net)
- D2 pad A: Net-(D1-PadA) -> (no net)
- R1 pad 1: Net-(D2-PadA) -> Net-(D1-PadA)
- R2 pad 1: Net-(D1-PadA) -> Net-(D2-PadA)
