File: PCB/donglev1-2025-02-02_151608/donglev1.kicad_sch (KiCad schematic)
At the start: 15 parts, among them J1 1734028-1, U1 CP2102N-24, U2 RYLR998

Commit message: other firmware testing
Parts:
- D1: renamed from D150060RS75000; value GREEN -> D1
- D2: renamed from D150060RS75000; value RED -> D2
- J1: footprint Adafruit CP2102N Friend:17340281 -> Connector_USB:USB_A_CNCTech_1001-011-01101_Horizontal
- U1: footprint Adafruit CP2102N Friend:QFN24_CP2102N_SIL -> Adafruit CP2102N Friend:QFN24_CP2102N_SIL-L
Changed lines of the file:
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@@
 		(on_board yes)
 		(dnp no)
-		(property "Reference" "D150060RS75000"
+		(property "Reference" "D2"
 			(at 184.785 80.01 0)
 			(effects
@@
 			)
 		)
-		(property "Value" "RED"
+		(property "Value" "D2"
 			(at 177.546 80.01 0)
 			(effects
@@
 			(project ""
 				(path "/c46daff7-deef-4110-b4a6-4ebe95bd77a0"
-					(reference "D150060RS75000")
+					(reference "D2")
 					(unit 1)
 				)
@@
 		(on_board yes)
 		(dnp no)
-		(property "Reference" "D150060RS75000"
+		(property "Reference" "D1"
 			(at 174.625 80.01 0)
 			(effects
@@
 			)
 		)
-		(property "Value" "GREEN"
+		(property "Value" "D1"
 			(at 167.386 80.01 0)
 			(effects
@@
 			(project ""
 				(path "/c46daff7-deef-4110-b4a6-4ebe95bd77a0"
-					(reference "D150060RS75000")
+					(reference "D1")
 					(unit 1)
 				)
@@
 			)
 		)
-		(property "Footprint" "Adafruit CP2102N Friend:QFN24_CP2102N_SIL"
+		(property "Footprint" "Adafruit CP2102N Friend:QFN24_CP2102N_SIL-L"
 			(at 134.62 93.98 0)
 			(effects
@@
 			)
 		)
-		(property "Footprint" "Adafruit CP2102N Friend:17340281"
+		(property "Footprint" "Connector_USB:USB_A_CNCTech_1001-011-01101_Horizontal"
 			(at 68.58 132.08 0)
 			(effects
